File: GPIB-USB.sch (KiCad schematic (older format))
At the start: 40 parts, among them J1 USB_B, J2 Conn_01x02, J3 Conn_ARM_JTAG_SWD_10, U1 LD1117S33CTR, U2 SN75160BDW, U3 WE-TVS-82400102, U4 FT230XQ, U5 SN75162BDW, U6 STM32F410RBTx, X1 112-024-113R001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

Commit message: update?
Parts:
- removed U4: FT230XQ, Package_DFN_QFN:QFN-16-1EP_4x4mm_P0.65mm_EP2.1x2.1mm, symbol Interface_USB:FT230XQ
- added U4: FT230XS, Package_SO:SSOP-16_3.9x4.9mm_P0.635mm, symbol Interface_USB:FT230XS
Connections:
- net +3V3: now also U4.3 (VCCIO)
- net +5V: now also U4.12 (VCC)
- net GND: now also U4.13 (GND), U4.5 (GND)
- net USART2_RX: now also U4.1 (TXD)
- net USART2_TX: now also U4.4 (RXD)
- net USB_ftdi_D+: now also U4.8 (USBDP)
- net USB_ftdi_D-: now also U4.9 (USBDM)
- new net +3.3VP: U4.10 (3V3OUT), U4.11 (~RESET)
- new net RXLED: U4.14 (CBUS1)
- new net TXLED: U4.7 (CBUS2)
- no-connect marks 2 -> 6
Changed lines of the file:
@@
 Wire Wire Line
 	4200 2800 4200 2750
-Wire Wire Line
-	4300 2750 4300 2800
 Connection ~ 4300 2800
 Wire Wire Line
@@
 Wire Wire Line
 	4300 2800 4300 2850
-$Comp
-L Interface_USB:FT230XQ U4
-U 1 1 5F3D7308
-P 4300 2050
-F 0 "U4" H 4600 1350 50  0000 C CNN
-F 1 "FT230XQ" H 4700 1450 50  0000 C CNN
-F 2 "Package_DFN_QFN:QFN-16-1EP_4x4mm_P0.65mm_EP2.1x2.1mm" H 5650 1450 50  0001 C CNN
-F 3 "https://www.ftdichip.com/Support/Documents/DataSheets/ICs/DS_FT230X.pdf" H 4300 2050 50  0001 C CNN
-	1    4300 2050
-	1    0    0    -1
-$EndComp
 $Comp
 L Device:R R1
@@
 P 4200 1350
 F 0 "#PWR015" H 4200 1200 50  0001 C CNN
-F 1 "+5V" H 4215 1523 50  0000 C CNN
+F 1 "+5V" H 4200 1500 50  0000 C CNN
 F 2 "" H 4200 1350 50  0001 C CNN
 F 3 "" H 4200 1350 50  0001 C CNN
@@
 P 4400 1350
 F 0 "#PWR016" H 4400 1200 50  0001 C CNN
-F 1 "+3.3V" H 4415 1523 50  0000 C CNN
+F 1 "+3.3V" H 4400 1500 50  0000 C CNN
 F 2 "" H 4400 1350 50  0001 C CNN
 F 3 "" H 4400 1350 50  0001 C CNN
@@
 Wire Wire Line
 	5000 1750 5250 1750
+$Comp
+L Interface_USB:FT230XS U4
+U 1 1 5F42777E
+P 4300 2050
+F 0 "U4" H 4700 1300 50  0000 C CNN
+F 1 "FT230XS" H 4750 1400 50  0000 C CNN
+F 2 "Package_SO:SSOP-16_3.9x4.9mm_P0.635mm" H 5300 1450 50  0001 C CNN
+F 3 "https://www.ftdichip.com/Support/Documents/DataSheets/ICs/DS_FT230X.pdf" H 4300 2050 50  0001 C CNN
+F 4 "FT230XS-R" H 4300 2050 50  0001 C CNN "article"
+	1    4300 2050
+	1    0    0    -1
+$EndComp
+Text GLabel 5000 2350 2    50   Input ~ 0
+TXLED
+Text GLabel 5000 2250 2    50   Input ~ 0
+RXLED
+NoConn ~ 5000 2150
+NoConn ~ 5000 2450
+NoConn ~ 5000 1850
+NoConn ~ 5000 1950
+$Comp
+L power:+3.3VP #PWR0101
+U 1 1 5F46E0D4
+P 3600 1650
+F 0 "#PWR0101" H 3750 1600 50  0001 C CNN
+F 1 "+3.3VP" V 3600 1800 50  0000 L CNN
+F 2 "" H 3600 1650 50  0001 C CNN
+F 3 "" H 3600 1650 50  0001 C CNN
+	1    3600 1650
+	0    -1   -1   0
+$EndComp
+$Comp
+L power:+3.3VP #PWR0102
+U 1 1 5F46FB28
+P 3600 2250
+F 0 "#PWR0102" H 3750 2200 50  0001 C CNN
+F 1 "+3.3VP" V 3600 2400 50  0000 L CNN
+F 2 "" H 3600 2250 50  0001 C CNN
+F 3 "" H 3600 2250 50  0001 C CNN
+	1    3600 2250
+	0    -1   -1   0
+$EndComp
 $EndSCHEMATC
