File: GPIB-USB.kicad_pcb (KiCad board)
At the start: 2 copper layers, 85 x 55 mm, 40 parts, among them J1 USB_B, J2 Conn_01x02, J3 Conn_ARM_JTAG_SWD_10, U1 LD1117S33CTR, U2 SN75160BDW, U3 WE-TVS-82400102, U4 FT230XQ, U5 SN75162BDW, U6 STM32F410RBTx, X1 112-024-113R001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

Commit message: update?
Parts:
- U4: value FT230XQ -> FT230XS; footprint Package_DFN_QFN:QFN-16-1EP_4x4mm_P0.65mm_EP2.1x2.1mm -> Package_SO:SSOP-16_3.9x4.9mm_P0.635mm
- moved R4 7.28 mm to (129.7, 112.8)
- moved U3 6.80 mm to (116.0, 81.8)
- moved R2 6.69 mm to (117.5, 77.8)
- moved R1 6.57 mm to (114.5, 77.8)
- moved R9 5.87 mm to (148.9, 79.1)
- moved C7 5.54 mm to (142.2, 117.8)
- moved C8 5.54 mm to (147.2, 117.8)
- moved Y1 5.54 mm to (144.7, 114.3)
- moved J3 4.91 mm to (137.2, 70.3)
- moved R3 4.91 mm to (132.2, 71.5)
- moved R5 4.91 mm to (137.9, 78.3)
- moved R6 4.91 mm to (140.2, 78.3)
- moved R7 4.91 mm to (135.7, 78.3)
- moved R8 4.91 mm to (142.4, 78.3)
- moved C1 4.46 mm to (120.8, 72.1), turned to 90 degrees
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Connections:
- net Net-(U4-Pad14) renamed RXLED
- U4 pad 1: +3V3 -> USART2_RX
- U4 pad 10: +5V -> +3.3VP
- U4 pad 11: Net-(U4-Pad11) -> +3.3VP
- U4 pad 12: Net-(U4-Pad12) -> +5V
- U4 pad 15: USART2_RX -> Net-(U4-Pad15)
- U4 pad 2: USART2_TX -> Net-(U4-Pad2)
- U4 pad 3: GND -> +3V3
- U4 pad 4: Net-(U4-Pad4) -> USART2_TX
- U4 pad 5: Net-(U4-Pad5) -> GND
- U4 pad 6: /USB_ftdi_D+ -> Net-(U4-Pad6)
- U4 pad 7: /USB_ftdi_D- -> TXLED
- U4 pad 8: Net-(U4-Pad8) -> /USB_ftdi_D+
- U4 pad 9: Net-(U4-Pad9) -> /USB_ftdi_D-
Routing:
- net Net-(FB1-Pad2): track 4.13 -> 34.5 mm
- net TCK: track 28.0 -> 2.25 mm
- net DIO5: track 25.2 -> 0.00 mm, vias 2 -> 0
- net VBUS: track 26.6 -> 1.50 mm
- net DIO6: track 24.5 -> 0.00 mm, vias 2 -> 0
- net DIO7: track 24.2 -> 0.00 mm, vias 2 -> 0
- net DIO8: track 23.4 -> 0.00 mm, vias 2 -> 0
- net DIO1: track 16.3 -> 0.00 mm
- net TMS: track 18.6 -> 2.25 mm
- net DIO2: track 15.6 -> 0.00 mm
- net conDAV: track 6.02 -> 21.6 mm, vias 0 -> 1
- net DIO3: track 14.9 -> 0.00 mm
- net +5V: track 18.2 -> 3.60 mm, vias 2 -> 1
- net DIO4: track 14.1 -> 0.00 mm
- net /CK-: track 14.1 -> 0.00 mm
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Other:
- board text added: "Solothurn - 2020"

Commit message: upgrade to Kicad6
Other:
- net class Default removed
